File: swarm.sch (KiCad schematic (older format))
At the start: 24 parts, among them P1 USB_OTG, P2 CONN_02X20, SW1 SW_PUSH, U1 STM32F103RETx, U2 LM3671MF-3.3, Y1 Crystal

Commit message: Replaces 0603 components with smaller fooprint Regenerated net file and imported in pcbnew
Parts:
- C1, C10, C11, C12, C13, C2, C3, C4, C5, C6, C7, C8, C9: footprint Capacitors_SMD:C_1206_HandSoldering -> Capacitors_SMD:C_1206
- P3: renamed from P?; footprint (none) -> Pin_Headers:Pin_Header_Angled_1x05
Changed lines of the file:
@@
 F 0 "C10" H 10225 1200 50  0000 L CNN
 F 1 "100n" H 10225 1000 50  0000 L CNN
-F 2 "Capacitors_SMD:C_1206_HandSoldering" H 10238 950 50  0001 C CNN
+F 2 "Capacitors_SMD:C_1206" H 10238 950 50  0001 C CNN
 F 3 "" H 10200 1100 50  0000 C CNN
 	1    10200 1100
@@
 F 0 "C11" H 10475 1200 50  0000 L CNN
 F 1 "100n" H 10475 1000 50  0000 L CNN
-F 2 "Capacitors_SMD:C_1206_HandSoldering" H 10488 950 50  0001 C CNN
+F 2 "Capacitors_SMD:C_1206" H 10488 950 50  0001 C CNN
 F 3 "" H 10450 1100 50  0000 C CNN
 	1    10450 1100
@@
 F 0 "C12" H 10725 1200 50  0000 L CNN
 F 1 "100n" H 10725 1000 50  0000 L CNN
-F 2 "Capacitors_SMD:C_1206_HandSoldering" H 10738 950 50  0001 C CNN
+F 2 "Capacitors_SMD:C_1206" H 10738 950 50  0001 C CNN
 F 3 "" H 10700 1100 50  0000 C CNN
 	1    10700 1100
@@
 F 0 "C13" H 10975 1200 50  0000 L CNN
 F 1 "100n" H 10975 1000 50  0000 L CNN
-F 2 "Capacitors_SMD:C_1206_HandSoldering" H 10988 950 50  0001 C CNN
+F 2 "Capacitors_SMD:C_1206" H 10988 950 50  0001 C CNN
 F 3 "" H 10950 1100 50  0000 C CNN
 	1    10950 1100
@@
 F 0 "C8" H 9725 1200 50  0000 L CNN
 F 1 "100n" H 9725 1000 50  0000 L CNN
-F 2 "Capacitors_SMD:C_1206_HandSoldering" H 9738 950 50  0001 C CNN
+F 2 "Capacitors_SMD:C_1206" H 9738 950 50  0001 C CNN
 F 3 "" H 9700 1100 50  0000 C CNN
 	1    9700 1100
@@
 F 0 "C9" H 9975 1200 50  0000 L CNN
 F 1 "100n" H 9975 1000 50  0000 L CNN
-F 2 "Capacitors_SMD:C_1206_HandSoldering" H 9988 950 50  0001 C CNN
+F 2 "Capacitors_SMD:C_1206" H 9988 950 50  0001 C CNN
 F 3 "" H 9950 1100 50  0000 C CNN
 	1    9950 1100
@@
 F 0 "C7" H 9275 1200 50  0000 L CNN
 F 1 "10u" H 9275 1000 50  0000 L CNN
-F 2 "Capacitors_SMD:C_1206_HandSoldering" H 9288 950 50  0001 C CNN
+F 2 "Capacitors_SMD:C_1206" H 9288 950 50  0001 C CNN
 F 3 "" H 9250 1100 50  0000 C CNN
 	1    9250 1100
@@
 F 0 "C6" H 8875 1200 50  0000 L CNN
 F 1 "1u" H 8875 1000 50  0000 L CNN
-F 2 "Capacitors_SMD:C_1206_HandSoldering" H 8888 950 50  0001 C CNN
+F 2 "Capacitors_SMD:C_1206" H 8888 950 50  0001 C CNN
 F 3 "" H 8850 1100 50  0000 C CNN
 	1    8850 1100
@@
 F 0 "C4" H 3875 3000 50  0000 L CNN
 F 1 "100n" H 3875 2800 50  0000 L CNN
-F 2 "Capacitors_SMD:C_1206_HandSoldering" H 3888 2750 50  0001 C CNN
+F 2 "Capacitors_SMD:C_1206" H 3888 2750 50  0001 C CNN
 F 3 "" H 3850 2900 50  0000 C CNN
 	1    3850 2900
@@
 F 0 "C3" H 3375 4650 50  0000 L CNN
 F 1 "C" H 3375 4450 50  0000 L CNN
-F 2 "Capacitors_SMD:C_1206_HandSoldering" H 3388 4400 50  0001 C CNN
+F 2 "Capacitors_SMD:C_1206" H 3388 4400 50  0001 C CNN
 F 3 "" H 3350 4550 50  0000 C CNN
 	1    3350 4550
@@
 F 0 "C5" H 3975 4650 50  0000 L CNN
 F 1 "C" H 3975 4450 50  0000 L CNN
-F 2 "Capacitors_SMD:C_1206_HandSoldering" H 3988 4400 50  0001 C CNN
+F 2 "Capacitors_SMD:C_1206" H 3988 4400 50  0001 C CNN
 F 3 "" H 3950 4550 50  0000 C CNN
 	1    3950 4550
@@
 F 0 "C1" H 1425 1300 50  0000 L CNN
 F 1 "10uF" H 1425 1100 50  0000 L CNN
-F 2 "Capacitors_SMD:C_1206_HandSoldering" H 1438 1050 50  0001 C CNN
+F 2 "Capacitors_SMD:C_1206" H 1438 1050 50  0001 C CNN
 F 3 "" H 1400 1200 50  0000 C CNN
 	1    1400 1200
@@
 F 0 "C2" H 3875 1400 50  0000 L CNN
 F 1 "22uF" H 3875 1200 50  0000 L CNN
-F 2 "Capacitors_SMD:C_1206_HandSoldering" H 3888 1150 50  0001 C CNN
+F 2 "Capacitors_SMD:C_1206" H 3888 1150 50  0001 C CNN
 F 3 "" H 3850 1300 50  0000 C CNN
 	1    3850 1300
@@
 Connection ~ 7450 6300
 Wire Wire Line
-	7450 6200 7450 6300
-Wire Wire Line
-	7450 6300 7450 6350
-Wire Wire Line
-	7250 2150 7350 2150
-Wire Wire Line
-	7350 2150 7450 2150
-Wire Wire Line
-	7450 2150 7550 2150
-Wire Wire Line
-	7550 2150 7650 2150
+	7450 6200 7450 6350
+Wire Wire Line
+	7250 2150 7650 2150
 Wire Wire Line
 	7650 2150 7650 2200
@@
 Connection ~ 7550 2150
 Wire Wire Line
-	7450 2100 7450 2150
-Wire Wire Line
-	7450 2150 7450 2200
+	7450 2100 7450 2200
 Wire Wire Line
 	7350 2200 7350 2150
@@
 	7250 2150 7250 2200
 Wire Wire Line
-	7250 6300 7350 6300
-Wire Wire Line
-	7350 6300 7450 6300
-Wire Wire Line
-	7450 6300 7550 6300
-Wire Wire Line
-	7550 6300 7650 6300
+	7250 6300 7650 6300
 Wire Wire Line
 	7650 6300 7650 6200
@@
 	9700 950  9700 850
 Wire Wire Line
-	9700 850  9950 850
-Wire Wire Line
-	9950 850  10200 850
-Wire Wire Line
-	10200 850  10350 850
-Wire Wire Line
-	10350 850  10450 850
-Wire Wire Line
-	10450 850  10700 850
-Wire Wire Line
-	10700 850  10950 850
+	9700 850  10950 850
 Wire Wire Line
 	10950 850  10950 950
@@
 	9700 1250 9700 1350
 Wire Wire Line
-	9700 1350 9950 1350
-Wire Wire Line
-	9950 1350 10200 1350
-Wire Wire Line
-	10200 1350 10350 1350
-Wire Wire Line
-	10350 1350 10450 1350
-Wire Wire Line
-	10450 1350 10700 1350
-Wire Wire Line
-	10700 1350 10950 1350
+	9700 1350 10950 1350
 Wire Wire Line
 	10950 1350 10950 1250
@@
 	3850 3050 3850 3250
 Wire Wire Line
-	3550 2600 3850 2600
-Wire Wire Line
-	3850 2600 4650 2600
+	3550 2600 4650 2600
 Wire Wire Line
 	3850 2600 3850 2750
@@
 	4650 3900 3350 3900
 Wire Wire Line
-	3350 3900 3350 4200
-Wire Wire Line
-	3350 4200 3350 4400
+	3350 3900 3350 4400
 Wire Wire Line
 	3350 4200 3550 4200
@@
 	3850 4200 3950 4200
 Wire Wire Line
-	3950 4000 3950 4200
-Wire Wire Line
-	3950 4200 3950 4400
+	3950 4000 3950 4400
 Wire Wire Line
 	3950 4750 3950 4700
@@
 Connection ~ 1400 1000
 Wire Wire Line
-	1400 1350 1400 1400
-Wire Wire Line
-	1400 1400 1400 1650
-Wire Wire Line
-	1400 1650 1400 1700
-Wire Wire Line
-	1200 1400 1400 1400
-Wire Wire Line
-	1400 1400 1650 1400
-Wire Wire Line
-	3850 750  3850 800
-Wire Wire Line
-	3850 800  3850 1000
-Wire Wire Line
-	3850 1000 3850 1100
-Wire Wire Line
-	3850 1100 3850 1150
+	1400 1350 1400 1700
+Wire Wire Line
+	1200 1400 1650 1400
+Wire Wire Line
+	3850 750  3850 1150
 Wire Wire Line
 	3050 1100 3850 1100
 Wire Wire Line
-	1400 750  1400 1000
-Wire Wire Line
-	1400 1000 1400 1050
+	1400 750  1400 1050
 Connection ~ 3850 1000
 Wire Wire Line
@@
 	3050 1200 3200 1200
 Wire Wire Line
-	1200 1000 1400 1000
-Wire Wire Line
-	1400 1000 1650 1000
+	1200 1000 1650 1000
 Connection ~ 3850 1100
 Wire Wire Line
@@
 LCD_RST
 $Comp
-L CONN_01X05 P?
+L CONN_01X05 P3
 U 1 1 584388C3
 P 950 4650
-F 0 "P?" H 950 4950 50  0000 C CNN
+F 0 "P3" H 950 4950 50  0000 C CNN
 F 1 "CONN_01X05" V 1050 4650 50  0000 C CNN
-F 2 "" H 950 4650 50  0000 C CNN
+F 2 "Pin_Headers:Pin_Header_Angled_1x05" H 950 4650 50  0001 C CNN
 F 3 "" H 950 4650 50  0000 C CNN
 	1    950  4650
